File: LEDCube.brd (EAGLE design)
At the start: 100.5 x 80.2 mm, 25 parts

Commit message: Routed PCB Array Board
Routing:
- net VCC: track 311.6 -> 0.00 mm, vias 1 -> 0
- net GND: track 216.1 -> 0.00 mm, vias 5 -> 0
- net UCA0CLK: track 126.4 -> 0.00 mm, vias 5 -> 0
- net RST2: track 124.9 -> 0.00 mm, vias 2 -> 0
- net SOMI: track 123.6 -> 0.00 mm, vias 6 -> 0
- net SIMO: track 105.5 -> 0.00 mm, vias 6 -> 0
- net RST4: track 92.1 -> 0.00 mm, vias 2 -> 0
- net RST3: track 84.5 -> 0.00 mm, vias 2 -> 0
- net 2C0: track 82.0 -> 0.00 mm, vias 1 -> 0
- net 1A2: track 77.5 -> 0.00 mm, vias 1 -> 0
- net 0C4: track 77.5 -> 0.00 mm, vias 1 -> 0
- net RST0: track 77.2 -> 0.00 mm, vias 2 -> 0
- net 0C1: track 74.7 -> 0.00 mm, vias 1 -> 0
- net 3A2: track 72.7 -> 0.00 mm, vias 1 -> 0
- net 1A0: track 72.2 -> 0.00 mm, vias 1 -> 0
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