File: CubePCB/LEDCube.brd (EAGLE design)
At the start: 100 x 80 mm, 55 parts

Commit message: Routed PCB Array Board
Parts:
- moved JP1 53.9 mm to (33.0, 16.0), turned to 0 degrees
- moved JP2 47.9 mm to (73.0, 16.0), turned to 0 degrees
- moved JP4 35.9 mm to (33.0, 52.0), turned to 0 degrees
- moved JP5 35.4 mm to (73.0, 52.0), turned to 0 degrees
- moved JP3 10.1 mm to (73.0, 33.1), turned to 0 degrees
Routing:
- net 1A5: track 0.00 -> 119.7 mm, vias 0 -> 1
- net 5A3: track 0.00 -> 117.5 mm
- net 1C5: track 0.00 -> 116.2 mm
- net 1A2: track 0.00 -> 114.8 mm
- net 5C2: track 0.00 -> 108.6 mm, vias 0 -> 1
- net 5A1: track 0.00 -> 107.2 mm, vias 0 -> 2
- net 4A5: track 0.00 -> 101.7 mm
- net 5C3: track 0.00 -> 101.1 mm, vias 0 -> 2
- net 5C1: track 0.00 -> 98.2 mm, vias 0 -> 2
- net 1C2: track 0.00 -> 97.2 mm
- net 5A4: track 0.00 -> 89.7 mm
- net 5A2: track 0.00 -> 88.8 mm, vias 0 -> 2
- net 1C3: track 0.00 -> 87.5 mm
- net 5C5: track 0.00 -> 84.7 mm, vias 0 -> 1
- net 5C4: track 0.00 -> 82.1 mm, vias 0 -> 1
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