File: MSPCube/LEDCube.brd (EAGLE design)
At the start: 100.5 x 80.2 mm, 25 parts

Commit message: printed version
Parts:
- moved JP1 60.7 mm to (32.8, 16.1)
- moved JP4 60.0 mm to (33.0, 52.0)
- moved JP5 27.0 mm to (72.8, 52.1)
- moved JP3 20.2 mm to (73.0, 33.1)
- moved JP2 20.0 mm to (73.0, 16.0)
- moved JP26 11.8 mm to (34.4, 34.2)
- moved JP22 4.23 mm to (70.0, 24.6)
- moved JP21 3.98 mm to (70.0, 7.65)
- moved JP24 3.28 mm to (70.4, 64.5)
- moved JP20 2.42 mm to (22.4, 76.3)
- moved JP23 2.37 mm to (70.2, 42.6)
- moved C1 2.09 mm to (18.0, 19.9)
- moved R2 0.21 mm to (9.99, 24.1)
Routing:
- net VCC: track 0.00 -> 228.9 mm, vias 0 -> 3
- net GND: track 0.00 -> 220.4 mm, vias 0 -> 4
- net SIMO: track 0.00 -> 143.8 mm, vias 0 -> 6
- net SOMI: track 0.00 -> 122.8 mm, vias 0 -> 6
- net UCA0CLK: track 0.00 -> 113.3 mm, vias 0 -> 6
- net RST3: track 0.00 -> 102.7 mm, vias 0 -> 1
- net RST4: track 0.00 -> 95.2 mm
- net RST2: track 0.00 -> 84.9 mm, vias 0 -> 1
- net RST1: track 0.00 -> 77.2 mm, vias 0 -> 1
- net RST0: track 0.00 -> 60.5 mm
- net STE4: track 0.00 -> 56.2 mm, vias 0 -> 2
- net 4C0: track 0.00 -> 50.4 mm, vias 0 -> 1
- net STE0: track 0.00 -> 49.2 mm, vias 0 -> 2
- net 2C2: track 0.00 -> 45.2 mm
- net 4C1: track 0.00 -> 44.6 mm, vias 0 -> 1
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